File: Eagle Files/Leak Detector 2B.brd (EAGLE design)
At the start: 98.3 x 81.8 mm, 22 parts, among them IC1 MCP6004, IC2 MCP6004, IC3 MCP6004, K2 HE751

Commit message: Eagle board files
Connections:
- removed net D12: IC2.8, U$1.D12
- net D10: now also IC2.8
Routing:
- net GND: track 0.00 -> 366.5 mm
- net +5V: track 0.00 -> 165.7 mm, vias 0 -> 1
- net BATHROOM: track 0.00 -> 160.7 mm
- net SCL: track 0.00 -> 151.7 mm, vias 0 -> 3
- net SDA: track 0.00 -> 142.5 mm, vias 0 -> 3
- net WASH_MACH: track 0.00 -> 115.7 mm, vias 0 -> 1
- net VTRIG: track 0.00 -> 114.3 mm
- net WATER_TANK: track 0.00 -> 102.4 mm
- net DISHWASHER: track 0.00 -> 89.5 mm, vias 0 -> 1
- net +3V3: track 0.00 -> 86.0 mm
- net SPARE1: track 0.00 -> 83.3 mm, vias 0 -> 1
- net SPARE2: track 0.00 -> 79.9 mm, vias 0 -> 2
- net D1: track 0.00 -> 76.3 mm
- net HOT_TUB_PUMP: track 0.00 -> 73.5 mm
- net N$4: track 0.00 -> 72.4 mm, vias 0 -> 1
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Other:
- board text added: "Leak Detector Base v2"
- board text removed: "Leak Detector Base v3"
