File: Eagle Files/Leak Detector 2B.sch (EAGLE design)
At the start: 22 parts, among them IC1 MCP6004, IC2 MCP6004, IC3 MCP6004, K2 HE751

Commit message: Eagle board files
Connections:
- removed net D12: IC2C.OUT, U$1.D12
- net D10: now also IC2C.OUT
Other:
- note added: "Don't use D10, it's needed as SS for Ethernet"
- note added: "Leak Detector V2 PCB is designed to fit in OKW enclosure B6504112"
- note added: "Leonardo Pinout A0 - Hot water tank A1 - Boiler A2 - Frig A3 - Dishwasher A4 - Bathroom A5 - Washing Machine D0 - LED Water Detected + Reed Relay D1 - OLED Reset D2-3 - I2C D4 - Reserved for SD Card D5 - Pad for future use D6 - Hot Tub Pump D7 - Hot Tub Rear D8 - Water tank in corner D9 - Kitchen Sink D10 - spare D11 - spare PanStamp Pinout D4 - LED PanStamp Rx A4 - I2C A5 - I2C"
- note removed: "Leak Detector v3 PCB is designed to fit in OKW enclosure B6504112"
- note removed: "Leonardo Pinout A0 - Hot water tank A1 - Boiler A2 - Frig A3 - Dishwasher A4 - Bathroom A5 - Washing Machine D0 - LED Water Detected + Reed Relay D1 - OLED Reset D2-3 - I2C D4 - Reserved for SD Card D5 - Pad for future use D6 - Hot Tub Pump D7 - Hot Tub Rear D8 - Water tank in corner D9 - Kitchen Sink D12 - spare D11 - spare PanStamp Pinout D4 - LED PanStamp Rx A4 - I2C A5 - I2C"
- note removed: "To Do: Add reverse polarity protection on input volts"
Changed lines of the file:
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@@
 D8 - Water tank in corner
 D9 - Kitchen Sink
-D12 - spare
+D10 - spare
 D11 - spare
 PanStamp Pinout
@@
 A4 - I2C
 A5 - I2C</text>
-<text x="55.88" y="243.84" size="5.08" layer="97" font="vector">Leak Detector v3
+<text x="55.88" y="243.84" size="5.08" layer="97" font="vector">Leak Detector V2
 PCB is designed to fit in OKW enclosure B6504112</text>
 <text x="137.16" y="78.74" size="1.778" layer="97">OLED Display</text>
@@
 <text x="247.65" y="155.956" size="1.4224" layer="97">For Red Water
 Warning LED</text>
-<text x="-86.36" y="254" size="2.1844" layer="97">To Do:
-Add reverse polarity protection on input volts</text>
+<text x="-96.52" y="43.18" size="1.778" layer="97">Don't use D10, it's needed as SS for Ethernet</text>
 </plain>
 <instances>
@@
 <instance part="GND25" gate="1" x="152.4" y="134.62" rot="R180"/>
 <instance part="GND26" gate="1" x="228.6" y="137.16"/>
-<instance part="GND28" gate="1" x="259.08" y="195.58"/>
+<instance part="GND28" gate="1" x="236.22" y="195.58"/>
 <instance part="GND30" gate="1" x="248.92" y="63.5"/>
 <instance part="P+2" gate="1" x="223.52" y="66.04" rot="MR270"/>
@@
 <pinref part="U$1" gate="G$1" pin="GND"/>
 <pinref part="GND28" gate="1" pin="GND"/>
-<wire x1="226.06" y1="198.12" x2="259.08" y2="198.12" width="0.1524" layer="91"/>
+<wire x1="226.06" y1="198.12" x2="236.22" y2="198.12" width="0.1524" layer="91"/>
 </segment>
 <segment>
@@
 <label x="231.14" y="187.96" size="1.778" layer="95" xref="yes"/>
 </segment>
+<segment>
+<wire x1="53.34" y1="129.54" x2="58.42" y2="129.54" width="0.1524" layer="91"/>
+<label x="58.42" y="129.54" size="1.778" layer="95" xref="yes"/>
+<pinref part="IC2" gate="C" pin="OUT"/>
+</segment>
 </net>
 <net name="D11" class="0">
@@
 </segment>
 </net>
-<net name="D12" class="0">
-<segment>
-<pinref part="U$1" gate="G$1" pin="D12"/>
-<wire x1="226.06" y1="193.04" x2="231.14" y2="193.04" width="0.1524" layer="91"/>
-<label x="231.14" y="193.04" size="1.778" layer="95" xref="yes"/>
-</segment>
-<segment>
-<wire x1="53.34" y1="129.54" x2="58.42" y2="129.54" width="0.1524" layer="91"/>
-<label x="58.42" y="129.54" size="1.778" layer="95" xref="yes"/>
-<pinref part="IC2" gate="C" pin="OUT"/>
-</segment>
-</net>
